File: pcbs/capacitive_plate_pcb/capacitive_plate_pcb.kicad_pcb (KiCad board)
At the start: 2 copper layers, 29 parts, among them J1 BM09B-SRSS-TB_LF__SN_, J2 SM08B-SRSS-TB_LF__SN_, U2 MCP1824T-3302E_OT, U3 ICM-42670-P

Commit message: almost done layout
Parts:
- added C16: 4.7uF, Capacitor_SMD:C_0603_1608Metric, B.Cu at (-70.2, -15.8)
- added JP2: Jumper_2_Bridged, Jumper:SolderJumper-2_P1.3mm_Bridged2Bar_RoundedPad1.0x1.5mm, B.Cu at (-51.4, 13.3)
- added R5: 10k, Capacitor_SMD:C_0603_1608Metric, B.Cu at (-62.1, -4.80)
- added R6: 10k, Capacitor_SMD:C_0603_1608Metric, B.Cu at (-64.9, -0.40)
- added R7: 10k, Capacitor_SMD:C_0603_1608Metric, B.Cu at (-70.2, -1.10)
- added R8: 100k, Capacitor_SMD:C_0603_1608Metric, B.Cu at (-73.2, -12.2)
- added REF**: touch_matrix_row, bjr_footprint_lib:touch_matrix_column, F.Cu at (3.50, 84.0)
- added REF**: touch_matrix_row, bjr_footprint_lib:touch_matrix_column_mod2, F.Cu at (24.5, 84.0)
- added REF**: touch_matrix_row, bjr_footprint_lib:touch_matrix_row, F.Cu at (-49.0, 73.5)
- added REF**: touch_matrix_row, bjr_footprint_lib:touch_matrix_column, F.Cu at (-10.5, 84.0)
- added REF**: touch_matrix_row, bjr_footprint_lib:touch_matrix_row, F.Cu at (-49.0, -80.5)
- added REF**: touch_matrix_row, bjr_footprint_lib:touch_matrix_row, F.Cu at (-49.0, -59.5)
- added REF**: touch_matrix_row, bjr_footprint_lib:touch_matrix_row, F.Cu at (-49.0, 24.5)
- added REF**: touch_matrix_row, bjr_footprint_lib:touch_matrix_column, F.Cu at (38.5, 84.0)
- added REF**: touch_matrix_row, bjr_footprint_lib:touch_matrix_row, F.Cu at (-49.0, 38.5)
- added REF**: touch_matrix_row, bjr_footprint_lib:touch_matrix_row, F.Cu at (-49.0, 31.5)
- added REF**: touch_matrix_row, bjr_footprint_lib:touch_matrix_column, F.Cu at (-17.5, 84.0)
- added REF**: touch_matrix_row, bjr_footprint_lib:touch_matrix_row, F.Cu at (-49.0, 66.5)
- added REF**: touch_matrix_row, bjr_footprint_lib:touch_matrix_column, F.Cu at (-38.5, 84.0)
- added REF**: touch_matrix_row, bjr_footprint_lib:touch_matrix_column, F.Cu at (-31.5, 84.0)
- added REF**: touch_matrix_row, bjr_footprint_lib:touch_matrix_row, F.Cu at (-49.0, -3.50)
- added REF**: touch_matrix_row, bjr_footprint_lib:touch_matrix_row, F.Cu at (-49.0, 52.5)
- added REF**: touch_matrix_row, bjr_footprint_lib:touch_matrix_row, F.Cu at (-49.0, -17.5)
- added REF**: touch_matrix_row, bjr_footprint_lib:touch_matrix_row, F.Cu at (-49.0, -73.5)
- added REF**: touch_matrix_row, bjr_footprint_lib:touch_matrix_row, F.Cu at (-49.0, 17.5)
- added REF**: touch_matrix_row, bjr_footprint_lib:touch_matrix_column, F.Cu at (-3.50, 84.0)
- added REF**: touch_matrix_row, bjr_footprint_lib:touch_matrix_row, F.Cu at (-49.0, -45.5)
- added REF**: touch_matrix_row, bjr_footprint_lib:touch_matrix_row, F.Cu at (-49.0, -52.5)
- added REF**: touch_matrix_row, bjr_footprint_lib:touch_matrix_column, F.Cu at (10.5, 84.0)
- added REF**: touch_matrix_row, bjr_footprint_lib:touch_matrix_row, F.Cu at (-49.0, -66.5)
- added REF**: touch_matrix_row, bjr_footprint_lib:touch_matrix_row, F.Cu at (-49.0, 59.5)
- added REF**: touch_matrix_row, bjr_footprint_lib:touch_matrix_row, F.Cu at (-49.0, 80.5)
- added REF**: touch_matrix_row, bjr_footprint_lib:touch_matrix_row, F.Cu at (-49.0, 3.50)
- added REF**: touch_matrix_row, bjr_footprint_lib:touch_matrix_row, F.Cu at (-49.0, 10.5)
- added REF**: touch_matrix_row, bjr_footprint_lib:touch_matrix_row, F.Cu at (-49.0, -38.5)
- added REF**: touch_matrix_row, bjr_footprint_lib:touch_matrix_column_mod1, F.Cu at (-24.5, 84.0)
- added REF**: touch_matrix_row, bjr_footprint_lib:touch_matrix_row, F.Cu at (-49.0, -31.5)
- added REF**: touch_matrix_row, bjr_footprint_lib:touch_matrix_row, F.Cu at (-49.0, 45.5)
- added REF**: touch_matrix_row, bjr_footprint_lib:touch_matrix_column, F.Cu at (45.5, 84.0)
- added REF**: touch_matrix_row, bjr_footprint_lib:touch_matrix_column, F.Cu at (31.5, 84.0)
- added REF**: touch_matrix_row, bjr_footprint_lib:touch_matrix_row, F.Cu at (-49.0, -24.5)
- added REF**: touch_matrix_row, bjr_footprint_lib:touch_matrix_row, F.Cu at (-49.0, -10.5)
- added REF**: touch_matrix_row, bjr_footprint_lib:touch_matrix_column, F.Cu at (17.5, 84.0)
- added REF**: touch_matrix_row, bjr_footprint_lib:touch_matrix_column, F.Cu at (-45.5, 84.0)
- added TP1: TestPoint, TestPoint:TestPoint_Pad_D1.5mm, B.Cu at (-66.4, -9.05)
- added TP2: TestPoint, TestPoint:TestPoint_Pad_D1.5mm, B.Cu at (-72.7, -8.15)
- added TP3: TestPoint, TestPoint:TestPoint_Pad_D1.5mm, B.Cu at (-74.0, -16.9)
- C1: value 1uF -> 10nF; moved to B.Cu
- C10: value 10nF -> 1uF; moved to B.Cu
- C11, C5: value 4.7uF -> 22nF; moved to B.Cu
- C12: value 4.7uF -> 10n; moved to B.Cu
- C13: value 100n -> 4.7uF; moved to B.Cu
- C14: value 2.2uF -> 100n; footprint Capacitor_SMD:C_0805_2012Metric -> Capacitor_SMD:C_0603_1608Metric; moved to B.Cu
- C15: value 10n -> 2.2uF; footprint Capacitor_SMD:C_0603_1608Metric -> Capacitor_SMD:C_0805_2012Metric; moved to B.Cu
- C2, J1, J2, M1, M2, M3, M4, R1: moved to B.Cu
- C3: value 100n -> 22nF; moved to B.Cu
- C4: value 100n -> 2.2nF; moved to B.Cu
- C6, C8: value 100n -> 2.2uF; footprint Capacitor_SMD:C_0603_1608Metric -> Capacitor_SMD:C_0805_2012Metric; moved to B.Cu
- C7: value 1uF -> 22nF; moved to B.Cu
- C9: value 10nF -> 22nF; moved to B.Cu
- JP1: value SolderJumper_3_Bridged12 -> SolderJumper_2_Open; footprint Jumper:SolderJumper-3_P2.0mm_Open_TrianglePad1.0x1.5mm_NumberLabels -> Jumper:SolderJumper-2_P1.3mm_Open_TrianglePad1.0x1.5mm; moved to B.Cu
- R2, R3: value 10k -> 47R; footprint Capacitor_SMD:C_0603_1608Metric -> Resistor_SMD:R_0603_1608Metric; moved to B.Cu
- R4: value 100k -> 47R; footprint Capacitor_SMD:C_0603_1608Metric -> Resistor_SMD:R_0603_1608Metric; moved to B.Cu
- U1: value ~ -> ATMXT336UD-MAUHA1; footprint bjr_footprint_lib:UFBGA-88_6x6mm_Layout11x11_P0.5mm -> bjr_footprint_lib:XQFN-56-1EP_6x6mm_P0.4mm_EP4.6x4.6mm_ThermalVias; moved to B.Cu
- U2: value MCP1824T-3302E_OT -> ICM-42670-P; footprint bjr_footprint_lib:SOT95P280X145-5N -> bjr_footprint_lib:IC_ICM-42670-P; moved to B.Cu
- U3: value ICM-42670-P -> MCP1824T-3302E_OT; footprint bjr_footprint_lib:IC_ICM-42670-P -> bjr_footprint_lib:SOT95P280X145-5N; moved to B.Cu
- moved J2 290.4 mm to (-80.2, 0.00), turned to 90 degrees
- moved U3 253.2 mm to (-70.2, -12.2), turned to 180 degrees
- moved JP1 248.9 mm to (-62.9, -10.1), turned to 180 degrees
- moved R4 242.8 mm to (-69.4, -5.30)
- moved U2 236.7 mm to (-68.6, 10.0), turned to 180 degrees
- moved C13 235.4 mm to (-66.7, -13.3), turned to -90 degrees
- moved R2 233.1 mm to (-69.4, -6.80)
- moved C14 229.2 mm to (-69.5, 12.3), turned to 180 degrees
- moved U1 229.0 mm to (-57.6, -0.85), turned to 180 degrees
- moved R1 228.7 mm to (-68.7, -1.10), turned to 90 degrees
- moved R3 228.2 mm to (-63.6, -4.80), turned to -90 degrees
- moved C11 227.0 mm to (-68.7, 2.40), turned to 90 degrees
- moved C9 226.3 mm to (-70.2, 1.90), turned to 90 degrees
- moved C15 226.1 mm to (-69.8, 14.1)
- moved C10 224.5 mm to (-67.2, 2.40), turned to -90 degrees
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Connections:
- C1 pad 1: GND -> /TOUCH_RST_BAR
- C1 pad 2: Net-(C1-Pad2) -> GND
- C10 pad 1: Net-(U1-EXTCAP1) -> Net-(U1-VDDCORE)
- C10 pad 2: Net-(U1-EXTCAP2) -> GND
- C11 pad 1: /+5V -> GND
- C11 pad 2: GND -> Net-(U1-VDDCORE)
- C13 pad 1: GND -> /+5V
- C13 pad 2: /+3.3V -> GND
- C14 pad 1: /+3.3V -> GND
- C14 pad 2: GND -> /+3.3V
- C2 pad 2: /+3.3V -> Net-(U1-XVDD)
- C3 pad 1: GND -> Net-(U1-XVDD)
- C3 pad 2: /+3.3V -> GND
- C4 pad 1: /+3.3V -> Net-(U1-EXTCAP1)
- C4 pad 2: GND -> Net-(U1-EXTCAP0)
- C6 pad 1: /+3.3V -> GND
- C6 pad 2: GND -> /+3.3V
- C7 pad 1: Net-(U1-VDDCORE) -> GND
- C7 pad 2: GND -> /+3.3V
- C8 pad 1: Net-(U1-VDDCORE) -> /+3.3V
- C9 pad 1: Net-(U1-EXTCAP0) -> GND
- C9 pad 2: Net-(U1-EXTCAP3) -> /+3.3V
- J1 pad S1: GND -> unconnected-(J1-SHIELD-PadS1)
- J1 pad S2: GND -> unconnected-(J1-SHIELD-PadS1)
- J2 pad 7: /TOUCH_RST_BAR -> Net-(J2-Pad7)
- J2 pad 8: /TOUCH_DBG_CLK -> Net-(J2-Pad8)
- J2 pad P1: (no net) -> unconnected-(J2-PadP1)
- J2 pad P2: (no net) -> unconnected-(J2-PadP2)
- JP1 pad 1: /+3.3V -> GND
- JP1 pad 2: Net-(JP1-C) -> Net-(JP1-B)
- R1 pad 2: Net-(U1-TEST_BAR) -> /TOUCH_RST_BAR
- R2 pad 1: /+3.3V -> Net-(J2-Pad8)
- R2 pad 2: /TOUCH_RST_BAR -> /TOUCH_DBG_CLK
- R3 pad 1: /+3.3V -> Net-(JP1-B)
- R3 pad 2: /TOUCH_CHG_BAR -> Net-(U1-GKEYY0/DBG_SS)
- R4 pad 1: /PWRGD -> Net-(J2-Pad7)
- R4 pad 2: /+3.3V -> /TOUCH_DBG_DATA
- U2 pad 1: /+5V -> GND
- U2 pad 2: GND -> unconnected-(U2-RESV_2-Pad2)
- U2 pad 3: /+5V -> unconnected-(U2-RESV_3-Pad3)
- U2 pad 4: /PWRGD -> /IMU_INT1
- U3 pad 1: GND -> /+5V
- U3 pad 2: unconnected-(U3-RESV_2-Pad2) -> GND
- U3 pad 3: unconnected-(U3-RESV_3-Pad3) -> /+5V
- U3 pad 4: /IMU_INT1 -> /PWRGD
Routing:
- net /DS0: track 0.00 -> 520.2 mm, vias 0 -> 7
- net GND: track 0.00 -> 180.0 mm, vias 0 -> 9
- net /+3.3V: track 0.00 -> 144.4 mm, vias 0 -> 1
- net /X13: track 0.00 -> 128.1 mm
- net /+5V: track 0.00 -> 123.4 mm, vias 0 -> 4
- net /X12: track 0.00 -> 121.0 mm
- net /TOUCH_RST_BAR: track 0.00 -> 115.9 mm, vias 0 -> 5
- net /TOUCH_CHG_BAR: track 0.00 -> 115.5 mm, vias 0 -> 5
- net /SCL: track 0.00 -> 115.5 mm, vias 0 -> 3
- net /X11: track 0.00 -> 113.8 mm
- net /SDA: track 0.00 -> 112.8 mm, vias 0 -> 3
- net /PWRGD: track 0.00 -> 110.5 mm, vias 0 -> 2
- net /X10: track 0.00 -> 110.2 mm
- net /X9: track 0.00 -> 98.7 mm
- net /X8: track 0.00 -> 91.7 mm
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- added copper zone on In2.Cu, net /PAS_SHIELD
- added copper zone on B.Cu, net GND
- added copper zone on F.Cu, net GND
Other:
- board outline added: 200 x 173.2 mm
- copper layers 2 -> 4
- board text added: "U1"
