File: pcbs/capacitive_plate_pcb/capacitive_plate_pcb.kicad_pcb (KiCad board)
At the start: 4 copper layers, 200 x 173.2 mm, 76 parts, among them J1 BM09B-SRSS-TB_LF__SN_, J2 SM08B-SRSS-TB_LF__SN_, U1 ATMXT336UD-MAUHA1, U2 ICM-42670-P, U3 MCP1824T-3302E_OT

Commit message: R01 plate pcb
Parts:
- added G***: LOGO, bjr_footprint_lib:EdBuilds_logo, B.Cu at (91.8, 0.00)
- R5, R6, R7, R8: footprint Capacitor_SMD:C_0603_1608Metric -> Resistor_SMD:R_0603_1608Metric
- moved C5 0.17 mm to (-53.4, -5.50)
Routing:
- net GND: track 180.0 -> 952.9 mm, vias 9 -> 20
- net /+3.3V: track 144.4 -> 61.0 mm, vias 1 -> 10
- net /Y23: track 86.7 -> 82.8 mm
- net /DS0: track 520.2 -> 517.4 mm
- net /IMU_INT1: track 72.6 -> 74.3 mm
- net /PWRGD: track 110.5 -> 112.0 mm
- net /+5V: track 123.4 -> 122.9 mm
- added copper zone on In1.Cu, net /+3.3V
- added copper zone on In2.Cu, net GND
- removed copper zone on B.Cu, net GND
- removed copper zone on F.Cu, net GND
Other:
- board text added: "+X"
- board text added: "+Y"
- board text added: "+Z"
- board text added: "BJR_01 Sensing Plate R01"
- board text removed: "U1"
