File: pcbs/capacitive_plate_pcb/capacitive_plate_pcb.kicad_sch (KiCad schematic)
At the start: 29 parts, among them J1 BM09B-SRSS-TB_LF__SN_, J2 SM08B-SRSS-TB_LF__SN_, U2 MCP1824T-3302E_OT, U3 ICM-42670-P

Commit message: almost done layout
Parts:
- removed C10: 10nF, Capacitor_SMD:C_0603_1608Metric, symbol Device:C
- removed C2: 1uF, Capacitor_SMD:C_0603_1608Metric, symbol Device:C
- removed JP1: SolderJumper_3_Bridged12, Jumper:SolderJumper-3_P2.0mm_Open_TrianglePad1.0x1.5mm_NumberLabels, symbol Jumper:SolderJumper_3_Bridged12
- removed U1: ~, bjr_footprint_lib:UFBGA-88_6x6mm_Layout11x11_P0.5mm, symbol bjr_symbol_lib:ATMXT640UD-CCUR001
- added C1: 10nF, Capacitor_SMD:C_0603_1608Metric, symbol Device:C
- added C11, C7: 22nF, Capacitor_SMD:C_0603_1608Metric, symbol Device:C
- added JP1: SolderJumper_2_Open, Jumper:SolderJumper-2_P1.3mm_Open_TrianglePad1.0x1.5mm, symbol Jumper:SolderJumper_2_Open
- added JP2: Jumper_2_Bridged, Jumper:SolderJumper-2_P1.3mm_Bridged2Bar_RoundedPad1.0x1.5mm, symbol Jumper:Jumper_2_Bridged
- added R2, R4: 47R, Resistor_SMD:R_0603_1608Metric, symbol Device:R
- added R5, R6: 10k, Capacitor_SMD:C_0603_1608Metric, symbol Device:R
- added TP1, TP2, TP3: TestPoint, TestPoint:TestPoint_Pad_D1.5mm, symbol Connector:TestPoint
- added U1: ATMXT336UD-MAUHA1, bjr_footprint_lib:XQFN-56-1EP_6x6mm_P0.4mm_EP4.6x4.6mm_ThermalVias, symbol bjr_symbol_lib:ATMXT336UD-MAUHA1
- C3: value 100n -> 22nF; Manufacturer number KAM15AR71H104KT -> KGM15AR71H223JT; Supplier code 581-KAM15AR71H104KT -> 581-KGM15AR71H223JT; Supplier website https://www.mouser.co.uk/ProductDetail/KYOCERA-AVX/KAM15AR7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 -> https://www.mouser.co.uk/ProductDetail/KYOCERA-AVX/KGM15AR7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
- C4: value 100n -> 2.2nF; Manufacturer number KAM15AR71H104KT -> KGM15AR71H222KT; Supplier code 581-KAM15AR71H104KT -> 581-KGM15AR71H222KT; Supplier website https://www.mouser.co.uk/ProductDetail/KYOCERA-AVX/KAM15AR7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 -> https://www.mouser.co.uk/ProductDetail/KYOCERA-AVX/KGM15AR7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
- C5: value 4.7uF -> 22nF; Manufacturer number 06033D475KAT2A -> KGM15AR71H223JT; Supplier code 581-06033D475KAT2A -> 581-KGM15AR71H223JT; Supplier website https://www.mouser.co.uk/ProductDetail/KYOCERA-AVX/06033D47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 -> https://www.mouser.co.uk/ProductDetail/KYOCERA-AVX/KGM15AR7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
- C6, C8: value 100n -> 2.2uF; footprint Capacitor_SMD:C_0603_1608Metric -> Capacitor_SMD:C_0805_2012Metric; Manufacturer number KAM15AR71H104KT -> 08053C225JAT2A; Supplier code 581-KAM15AR71H104KT -> 581-08053C225JAT2A; Supplier website https://www.mouser.co.uk/ProductDetail/KYOCERA-AVX/KAM15AR7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 -> https://www.mouser.co.uk/ProductDetail/KYOCERA-AVX/08053C22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
- C9: value 10nF -> 22nF; Manufacturer number KGM15AR71H103KT -> KGM15AR71H223JT; Supplier code 581-KGM15AR71H103KT -> 581-KGM15AR71H223JT; Supplier website https://www.mouser.co.uk/ProductDetail/KYOCERA-AVX/KGM15AR71H103KT?qs=Jm2GQyTW%2Fbg6jbH8a6Ap5w%3D%3D -> https://www.mouser.co.uk/ProductDetail/KYOCERA-AVX/KGM15AR71H223JT?qs=Jm2GQyTW%2Fbig4dazQ2H7jw%3D%3D
- R3: value 10k -> 47R; footprint Capacitor_SMD:C_0603_1608Metric -> Resistor_SMD:R_0603_1608Metric; Manufacturer Panasonic -> ROHM Semiconductor; Manufacturer number ERJ-3EKF1002V -> SDR03EZPF47R0; Supplier code 667-ERJ-3EKF1002V -> 755-SDR03EZPF47R0; Supplier website https://www.mouser.co.uk/ProductDetail/Panasonic/ERJ-3EKF10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 -> https://www.mouser.co.uk/ProductDetail/ROHM-Semiconductor/S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
- renumbered C7 to C10, C15 to C12, C11 to C13, C13 to C14, C14 to C15, C12 to C16, C1 to C2, M4 to M1, M3 to M2, M2 to M3, M1 to M4, R2 to R1, R1 to R7, R4 to R8, U3 to U2, U2 to U3
Connections:
- net +3.3V: now also C6.2, C8.1, C9.2, C7.2, R5.1, R6.1, TP3.1, U1.30 (VDD), U1.32 (VDDIO), U1.56 (AVDD); no longer C3.2, C4.1, C6.1, R3.1
- net +5V: now also TP1.1
- net GND: now also C3.2, C6.1, C9.1, U2.6 (GND), C1.2, C11.1, C7.1, JP1.1 (A), JP2.1 (A), U1.57 (GND); no longer C3.1, C4.2, C6.2, J1.S1 (SHIELD), J1.S2 (SHIELD)
- net PWRGD: now also TP2.1
- net SCL: now also U1.35 (SCL)
- net SDA: now also U1.34 (SDA)
- net TOUCH_CHG_BAR: now also R7.2, U1.37 (CHG_BAR); no longer R3.2
- net TOUCH_DBG_CLK: now also R2.2, U1.39 (DBG_CLK); no longer J2.8
- net TOUCH_DBG_DATA: now also R4.2, U1.38 (SYNC/DBG_DATA)
- net TOUCH_RST_BAR: now also C1.1, U1.36 (RESET_BAR); no longer J2.7
- net at C2.2: now also C3.1, U1.15 (XVDD)
- net at C10.1: now also C11.2, U1.31 (VDDCORE); no longer C8.1
- new net: J2.8, R2.1
- new net: J2.7, R4.1
- new net: R6.2, U1.33 (TEST_BAR)
- new net: R3.2, R5.2, U1.41 (GKEYY0/DBG_SS)
- new net: C4.1, U1.16 (EXTCAP1)
- new net: C4.2, U1.29 (EXTCAP0)
- new net: JP1.2 (B), R3.1
- new net: J1.S1 (SHIELD), J1.S2 (SHIELD)
- new net DS0: U1.40 (DS0)
- new net PAS_SHIELD: JP2.2 (B)
- new net X0: U1.1 (X0)
- new net X1: U1.2 (X1)
- new net X10: U1.11 (X10)
- new net X11: U1.12 (X11)
- new net X12: U1.13 (X12)
- new net X13: U1.14 (X13)
- new net X2: U1.3 (X2)
- new net X3: U1.4 (X3)
- new net X4: U1.5 (X4)
- new net X5: U1.6 (X5)
- new net X6: U1.7 (X6)
- new net X7: U1.8 (X7)
- new net X8: U1.9 (X8)
- new net X9: U1.10 (X9)
- new net Y0: U1.55 (Y0)
- new net Y1: U1.54 (Y1)
- new net Y10: U1.45 (Y10)
- new net Y11: U1.44 (Y11)
- new net Y12: U1.17 (Y12)
- new net Y13: U1.18 (Y13)
- new net Y14: U1.19 (Y14)
- new net Y15: U1.20 (Y15)
- new net Y16: U1.21 (Y16)
- new net Y17: U1.22 (Y17)
- new net Y18: U1.23 (Y18)
- new net Y19: U1.24 (Y19)
- new net Y2: U1.53 (Y2)
- new net Y20: U1.25 (Y20)
- new net Y21: U1.26 (Y21)
- new net Y22: U1.27 (Y22)
- new net Y23: U1.28 (Y23)
- new net Y3: U1.52 (Y3)
- new net Y4: U1.51 (Y4)
- new net Y5: U1.50 (Y5)
- new net Y6: U1.49 (Y6)
- new net Y7: U1.48 (Y7)
- new net Y8: U1.47 (Y8)
- new net Y9: U1.46 (Y9)
- no-connect marks 12 -> 10
Other:
- moved on the sheet: C2, R1, R7

Commit message: R01 plate pcb
Parts:
- J1: Availability In Stock -> (none); Check_prices https://www.snapeda.com/parts/BM09B-SRSS-TB(LF)(SN)/JST+Sal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 -> (none); MANUFACTURER JST Sales America Inc. -> (none); MAXIMUM_PACKAGE_HEIGHT 6.3 mm -> (none); MF JST Sales -> (none); MP BM09B-SRSS-TB(LF)(SN) -> (none); Manufacturer (none) -> JST; Manufacturer number (none) -> BM09B-SRSS-TB(LF)(SN); PARTREV N/A -> (none); Package None -> (none); Price None -> (none); SNAPEDA_PN BM09B-SRSS-TB(LF)(SN) -> (none); STANDARD Manufacturer Recommendations -> (none); SnapEDA_Link https://www.snapeda.com/parts/BM09B-SRSS-TB(LF)(SN)/JST+Sal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 -> (none); Supplier (none) -> Farnell; Supplier code (none) -> 1679135; Supplier website (none) -> https://uk.farnell.com/jst-japan-solderless-terminals/bm09b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
- J2: Availability In Stock -> (none); Check_prices https://www.snapeda.com/parts/SM08B-SRSS-TB(LF)(SN)/JST+Sal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 -> (none); MANUFACTURER JST -> (none); MF JST Sales -> (none); MP SM08B-SRSS-TB(LF)(SN) -> (none); Manufacturer (none) -> JST; Manufacturer number (none) -> SM08B-SRSS-TB(LF)(SN); Package None -> (none); Price None -> (none); SnapEDA_Link https://www.snapeda.com/parts/SM08B-SRSS-TB(LF)(SN)/JST+Sal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 -> (none); Supplier (none) -> Farnell; Supplier code (none) -> 1679124; Supplier website (none) -> https://uk.farnell.com/jst-japan-solderless-terminals/sm08b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
- M1, M2, M3, M4: Manufacturer (none) -> Wurth electronik; Manufacturer number (none) -> 9774010151R; Supplier (none) -> Farnell; Supplier code (none) -> 2766287; Supplier website (none) -> https://uk.farnell.com/wurth-elektronik/9774010151r/standof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
- R5, R6, R7, R8: footprint Capacitor_SMD:C_0603_1608Metric -> Resistor_SMD:R_0603_1608Metric
- U1: Manufacturer (none) -> Microchip Technology; Manufacturer number (none) -> ATMXT336UD-MAUHA1; Supplier (none) -> DigiKey; Supplier code (none) -> 150-ATMXT336UD-MAUHA1-ND; Supplier website (none) -> https://www.digikey.co.uk/en/products/detail/microchip-tech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
- U2: Availability In Stock -> (none); Check_prices https://www.snapeda.com/parts/ICM-42670-P/TDK+InvenSense/vi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 -> (none); MF TDK InvenSense -> (none); MP ICM-42670-P -> (none); Manufacturer (none) -> TDK InvenSense; Manufacturer number (none) -> ICM-42670-P; Package None -> (none); Price None -> (none); Purchase-URL https://www.snapeda.com/api/url_track_click_mouser/?unipart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 -> (none); SnapEDA_Link https://www.snapeda.com/parts/ICM-42670-P/TDK+InvenSense/vi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 -> (none); Supplier (none) -> Mouser; Supplier code (none) -> 410-ICM-42670-P; Supplier website (none) -> https://www.mouser.co.uk/ProductDetail/TDK-InvenSense/ICM-4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
- U3: Availability In Stock -> (none); MF Microchip -> (none); MP MCP1824T-3302E/OT -> (none); Manufacturer (none) -> Microchip; Manufacturer number (none) -> MCP1824T-3302E/OT; Price None -> (none); Supplier (none) -> Mouser; Supplier code (none) -> 579-MCP1824T-3302EOT; Supplier website (none) -> https://www.mouser.co.uk/ProductDetail/Microchip-Technology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
Other:
- moved on the sheet: C12, C13, C14, C15, C16, J1, JP2, R8, TP1, TP2, TP3, U2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
