File: pcbs/resistive_plate/resistive_plate.kicad_sch (KiCad schematic)
At the start: 21 parts, among them IC1 TSC2046EIPWR, IC2 LSM6DS3TR-C, J1 SFW4R-1STE1HLF, J2 BM08B-SRSS-TBT_LF__SN_, M10 1.1 mm, M11 1.1 mm, M12 1.1 mm, M5 1.1 mm, M6 1.1 mm, M7 1.1 mm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

Commit message: post mgf commit
Parts:
- M1, M2, M3, M4: Supplier (none) -> Mouser; Supplier_code (none) -> 710-9774010151R; Supplier_url (none) -> https://www.mouser.co.uk/ProductDetail/Wurth-Elektronik/977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
Other:
- moved on the sheet: M10, M11, M12, M5, M6, M7, M8, M9
