File: pcbs/reduced_resistive_board/reduced_resistive_board.kicad_sch (KiCad schematic)
At the start: 6 parts, among them IC1 TSC2046EIPWR, J1 SFW4R-1STE1HLF, J3 SM08B-SRSS-TB_LF__SN_

Commit message: STAGING
Parts:
- added C3, C6: 1uF, Capacitor_SMD:C_0603_1608Metric, symbol Device:C
- added C5: 0.1uF, Capacitor_SMD:C_0603_1608Metric, symbol Device:C
- added U1: ~, Package_TO_SOT_SMD:SOT-23-5, symbol bjr_symbol_lib:LD3985M28R
Connections:
- net GND: now also C3.2, C5.2, C6.2, U1.2 (GND)
- net VDD: now also C3.1, U1.1 (V_I), U1.3 (V_INH); no longer C1.1, C2.1, C4.1, IC1.1 (+VCC), IC1.10 (IOVDD)
- new net: C5.1, U1.4 (BYPASS)
- new net +2V8: C1.1, C2.1, C4.1, C6.1, IC1.1 (+VCC), IC1.10 (IOVDD), U1.5 (V_O)
