File: pcbs/reduced_resistive_board/reduced_resistive_board.kicad_pcb (KiCad board)
At the start: 2 copper layers, 26 x 25 mm, 11 parts, among them IC1 TSC2046EIPWR, J1 SFW4R-1STE1HLF, J3 SM08B-SRSS-TB_LF__SN_

Commit message: STAGING
Parts:
- added C3: 1uF, Capacitor_SMD:C_0603_1608Metric, F.Cu at (-7.16, 23.4)
- added C5: 0.1uF, Capacitor_SMD:C_0603_1608Metric, F.Cu at (-4.26, 25.9)
- added C6: 1uF, Capacitor_SMD:C_0603_1608Metric, F.Cu at (-1.46, 23.4)
- added U1: ~, Package_TO_SOT_SMD:SOT-23-5, F.Cu at (-4.30, 23.4)
- moved C1 2.78 mm to (-1.41, 28.8)
- moved C2 2.78 mm to (-3.70, 28.8)
- moved C4 2.78 mm to (7.23, 26.5)
- moved IC1 2.78 mm to (2.90, 26.9)
- moved J1 2.00 mm to (0.00, 37.5)
- moved J3 1.03 mm to (0.00, 14.3)
Connections:
- C1 pad 1: VDD -> +2V8
- C2 pad 1: VDD -> +2V8
- C4 pad 1: VDD -> +2V8
- IC1 pad 1: VDD -> +2V8
- IC1 pad 10: VDD -> +2V8
Routing:
- net +2V8: track 0.00 -> 33.9 mm, vias 0 -> 3
- net VDD: track 35.9 -> 12.0 mm, vias 3 -> 0
- net /SCK: track 15.0 -> 6.44 mm, vias 0 -> 2
- net GND: track 13.8 -> 17.3 mm, vias 3 -> 6
- net /CS_TOUCH: track 2.59 -> 5.99 mm
- net /MISO: track 2.61 -> 5.97 mm
- net /MOSI: track 2.73 -> 5.84 mm
- net Net-(U1-BYPASS): track 0.00 -> 1.63 mm
- net /X+: track 3.97 -> 5.56 mm
- net /Y+: track 3.82 -> 5.42 mm
- net /X-: track 3.95 -> 5.27 mm
- net /Y-: track 4.09 -> 5.13 mm
Other:
- board text added: "RRB R02"
- board text removed: "RRB R01"

Commit message: update but not sure what
Routing:
- net +2V8: track 33.9 -> 35.7 mm
Changed lines of the file:
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@@
 		(sheetfile "reduced_resistive_board.kicad_sch")
 		(attr smd)
-		(fp_line
-			(start -4.9 -2.75)
-			(end -3.17 -2.75)
-			(stroke
-				(width 0.127)
-				(type solid)
-			)
-			(layer "F.SilkS")
-		)
-		(fp_line
-			(start -4.9 2.75)
-			(end -4.9 -2.75)
-			(stroke
-				(width 0.127)
-				(type solid)
-			)
-			(layer "F.SilkS")
-		)
-		(fp_line
-			(start 3.17 -2.75)
-			(end 4.9 -2.75)
-			(stroke
-				(width 0.127)
-				(type solid)
-			)
-			(layer "F.SilkS")
-		)
-		(fp_line
-			(start 4.9 -2.75)
-			(end 4.9 2.75)
-			(stroke
-				(width 0.127)
-				(type solid)
-			)
-			(layer "F.SilkS")
-		)
-		(fp_line
-			(start 4.9 2.75)
-			(end -4.9 2.75)
-			(stroke
-				(width 0.127)
-				(type solid)
-			)
-			(layer "F.SilkS")
-		)
 		(fp_circle
 			(center -1.5 -4.85)
@@
 	)
 	(segment
-		(start 4.9915 24.1085)
-		(end 5.1 24)
-		(width 0.25)
-		(layer "F.Cu")
-		(net 3)
-	)
-	(segment
 		(start -7.1625 22.575)
 		(end -7.1625 22.1625)
@@
 	)
 	(segment
-		(start -1.4625 25.1865)
-		(end -1.449 25.2)
-		(width 0.25)
-		(layer "F.Cu")
-		(net 7)
-	)
-	(segment
 		(start -3.696 27.7945)
 		(end -1.41 27.7945)
@@
 	)
 	(segment
+		(start -2.702851 23.35)
+		(end -1.927851 24.125)
+		(width 0.25)
+		(layer "F.Cu")
+		(net 7)
+	)
+	(segment
 		(start -1.41 27.7945)
 		(end 2.819 27.7945)
@@
 	)
 	(segment
+		(start -1.927851 24.125)
+		(end -1.4625 24.125)
+		(width 0.25)
+		(layer "F.Cu")
+		(net 7)
+	)
+	(segment
 		(start -5.4375 23.4)
 		(end -6.385784 23.4)
@@
 	)
 	(segment
-		(start -1.4625 24.125)
-		(end -1.4625 25.1865)
-		(width 0.25)
-		(layer "F.Cu")
-		(net 7)
-	)
-	(segment
 		(start -5.0375 25.85)
 		(end -6.099 25.85)
@@
 	)
 	(via
-		(at -1.449 25.2)
+		(at -2.702851 23.35)
 		(size 0.8)
 		(drill 0.4)
@@
 	(segment
 		(start 0.062 23.962)
-		(end 0 23.9)
-		(width 0.25)
-		(layer "F.Cu")
-		(net 17)
-	)
-	(segment
-		(start 0.625 23.962)
-		(end 0.062 23.962)
+		(end 0.625 23.962)
 		(width 0.25)
 		(layer "F.Cu")
@@
 	)
 	(segment
+		(start -0.013856 23.542169)
+		(end -0.013856 23.886144)
+		(width 0.25)
+		(layer "F.Cu")
+		(net 17)
+	)
+	(segment
 		(start 1.5 20.247194)
 		(end 1.5 19.125)
@@
 		(net 17)
 	)
+	(segment
+		(start -0.013856 23.886144)
+		(end 0.062 23.962)
+		(width 0.25)
+		(layer "F.Cu")
+		(net 17)
+	)
 	(via
-		(at 0 23.9)
+		(at -0.013856 23.542169)
 		(size 0.8)
 		(drill 0.4)
@@
 	)
 	(segment
-		(start 0 23.9)
-		(end 0.355654 23.544346)
+		(start -0.013856 23.542169)
+		(end 0.355654 23.172659)
 		(width 0.25)
 		(layer "B.Cu")
@@
 	)
 	(segment
-		(start 0.355654 23.544346)
-		(end 0.355654 22.844346)
+		(start 1.976403 21.223597)
+		(end 1.976403 20.723597)
 		(width 0.25)
 		(layer "B.Cu")
@@
 	)
 	(segment
-		(start 1.976403 21.223597)
-		(end 1.976403 20.723597)
+		(start 0.355654 22.844346)
+		(end 1.976403 21.223597)
 		(width 0.25)
 		(layer "B.Cu")
@@
 	)
 	(segment
-		(start 0.355654 22.844346)
-		(end 1.976403 21.223597)
+		(start 0.355654 23.172659)
+		(end 0.355654 22.844346)
 		(width 0.25)
 		(layer "B.Cu")
@@
 	)
 	(segment
+		(start -5.423 24.423)
+		(end -5.423 26.10072)
+		(width 0.25)
+		(layer "B.Cu")
+		(net 22)
+	)
+	(segment
+		(start -3.6 22.6)
+		(end -5.423 24.423)
+		(width 0.25)
+		(layer "B.Cu")
+		(net 22)
+	)
+	(segment
 		(start 2.797597 19.997597)
 		(end 7.3 24.5)
@@
 	)
 	(segment
-		(start -1.571277 22.6)
-		(end -4.367 25.395723)
+		(start -0.349 22.6)
+		(end -3.6 22.6)
 		(width 0.25)
 		(layer "B.Cu")
@@
 	)
 	(segment
+		(start -5.84828 26.526)
+		(end -5.9 26.526)
+		(width 0.25)
+		(layer "B.Cu")
+		(net 22)
+	)
+	(segment
+		(start -5.9 29.1)
+		(end -5.1 29.9)
+		(width 0.25)
+		(layer "B.Cu")
+		(net 22)
+	)
+	(segment
+		(start -5.9 26.526)
+		(end -5.9 29.1)
+		(width 0.25)
+		(layer "B.Cu")
+		(net 22)
+	)
+	(segment
 		(start -4.987855 30.012145)
 		(end -5.1 29.9)
@@
 	)
 	(segment
-		(start -4.367 29.167)
-		(end -5.1 29.9)
+		(start 7.3 24.5)
+		(end 7.3 24.7)
 		(width 0.25)
 		(layer "B.Cu")
@@
 	)
 	(segment
-		(start 7.3 24.5)
-		(end 7.3 24.7)
+		(start -5.423 26.10072)
+		(end -5.84828 26.526)
 		(width 0.25)
 		(layer "B.Cu")
-		(net 22)
-	)
-	(segment
-		(start -4.367 25.395723)
-		(end -4.367 29.167)
-		(width 0.25)
-		(layer "B.Cu")
-		(net 22)
-	)
-	(segment
-		(start -0.349 22.6)
-		(end -1.571277 22.6)
-		(width 0.25)
-		(layer "B.Cu")
